Commit message: edits made

File: description/robot_core.xacro (robot description, xacro)
@@ -17,5 +17,5 @@
     <link name="body">
         <visual>
-            <origin xyz="0.15 0 0.75" />
+            <origin xyz="0.15 0 0.075" />
             <geometry>
                 <box size="0.3 0.3 0.15" />

Commit message: edits made

File: description/robot_core.xacro (robot description, xacro)
@@ -15,4 +15,9 @@
     <link name="base_link">
     </link>
+    <joint name="body_joint" type="fixed">
+        <parent link="base_link" />
+        <child link="body" />
+        <origin xyz="-0.1 0 0">
+    </joint>
     <link name="body">
         <visual>
@@ -24,8 +29,3 @@
         </visual>
     </link>
-    <joint name="body_joint" type="fixed">
-        <parent link="base_link" />
-        <child link="body" />
-        <origin xyz="-0.1 0 0">
-    </joint>
 </robot>
